File: Atmega328p_board.kicad_pcb (KiCad board)
At the start: 2 copper layers, 48.2 x 30.3 mm, 29 parts, among them J1 Conn_01x04_Pin, J2 Conn_01x04_Pin, J3 Conn_01x09_Pin, J4 Conn_02x03_Odd_Even, U1 24LC1025, U2 24LC1025, U3 ATMEGA328P-AU, U4 DS1337S_, Y1 16MHz, Y2 32.768 KHz

Commit message: Refined some routes
Routing:
- net /RESET: track 39.5 -> 38.8 mm
Changed lines of the file:
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@@
   (segment (start 163.5608 89.4944) (end 162.3568 88.2904) (width 0.25) (layer "F.Cu") (net 10))
   (segment (start 134.143 98.044) (end 133.158 98.044) (width 0.25) (layer "F.Cu") (net 10))
-  (segment (start 135.668 86.671582) (end 133.807018 84.8106) (width 0.25) (layer "F.Cu") (net 10))
+  (segment (start 133.2078 90.068401) (end 133.693001 89.5832) (width 0.25) (layer "F.Cu") (net 10))
   (segment (start 132.5728 83.2866) (end 133.1062 82.7532) (width 0.25) (layer "F.Cu") (net 10))
-  (segment (start 133.2078 90.068401) (end 133.693001 89.5832) (width 0.25) (layer "F.Cu") (net 10))
   (segment (start 156.1694 84.5312) (end 156.4488 84.8106) (width 0.25) (layer "F.Cu") (net 10))
   (segment (start 143.91 84.122) (end 142.8206 83.0326) (width 0.25) (layer "F.Cu") (net 10))
-  (segment (start 132.5728 84.8106) (end 132.5728 83.2866) (width 0.25) (layer "F.Cu") (net 10))
+  (segment (start 133.1062 82.7532) (end 134.493 82.7532) (width 0.25) (layer "F.Cu") (net 10))
   (segment (start 159.2663 96.5283) (end 164.8968 102.1588) (width 0.25) (layer "F.Cu") (net 10))
   (segment (start 133.2078 91.5416) (end 133.2078 90.068401) (width 0.25) (layer "F.Cu") (net 10))
   (segment (start 134.518 97.669) (end 134.143 98.044) (width 0.25) (layer "F.Cu") (net 10))
-  (segment (start 133.1062 82.7532) (end 134.493 82.7532) (width 0.25) (layer "F.Cu") (net 10))
   (segment (start 155.8138 84.5312) (end 156.1694 84.5312) (width 0.25) (layer "F.Cu") (net 10))
+  (segment (start 133.3684 86.3682) (end 132.5728 85.5726) (width 0.25) (layer "F.Cu") (net 10))
+  (segment (start 135.668 86.671582) (end 135.364618 86.3682) (width 0.25) (layer "F.Cu") (net 10))
   (segment (start 159.2663 94.5896) (end 160.259301 94.5896) (width 0.25) (layer "F.Cu") (net 10))
   (segment (start 156.4488 87.6046) (end 156.4488 84.8106) (width 0.25) (layer "F.Cu") (net 10))
@@
   (segment (start 160.259301 94.5896) (end 163.5608 91.288101) (width 0.25) (layer "F.Cu") (net 10))
   (segment (start 156.1694 84.5312) (end 156.4488 84.5312) (width 0.25) (layer "F.Cu") (net 10))
+  (segment (start 134.493 89.5832) (end 135.6742 89.5832) (width 0.25) (layer "F.Cu") (net 10))
   (segment (start 154.1885 84.5312) (end 154.4809 84.5312) (width 0.25) (layer "F.Cu") (net 10))
-  (segment (start 135.668 89.577) (end 135.668 86.671582) (width 0.25) (layer "F.Cu") (net 10))
   (segment (start 156.4488 84.6836) (end 156.4488 84.5312) (width 0.25) (layer "F.Cu") (net 10))
   (segment (start 159.2663 94.5896) (end 159.2663 96.5283) (width 0.25) (layer "F.Cu") (net 10))
   (segment (start 134.7724 83.0326) (end 134.493 82.7532) (width 0.25) (layer "F.Cu") (net 10))
   (segment (start 156.4488 84.5312) (end 156.7282 84.5312) (width 0.25) (layer "F.Cu") (net 10))
-  (segment (start 133.807018 84.8106) (end 132.5728 84.8106) (width 0.25) (layer "F.Cu") (net 10))
   (segment (start 143.91 84.857) (end 143.91 84.122) (width 0.25) (layer "F.Cu") (net 10))
+  (segment (start 132.5728 85.5726) (end 132.5728 83.2866) (width 0.25) (layer "F.Cu") (net 10))
   (segment (start 156.4488 84.8106) (end 156.4488 84.6836) (width 0.25) (layer "F.Cu") (net 10))
   (segment (start 143.91 85.6068) (end 144.7648 86.4616) (width 0.25) (layer "F.Cu") (net 10))
   (segment (start 156.4488 84.6836) (end 156.5758 84.6836) (width 0.25) (layer "F.Cu") (net 10))
   (segment (start 133.693001 89.5832) (end 134.493 89.5832) (width 0.25) (layer "F.Cu") (net 10))
+  (segment (start 135.668 89.577) (end 135.668 86.671582) (width 0.25) (layer "F.Cu") (net 10))
+  (segment (start 135.364618 86.3682) (end 133.3684 86.3682) (width 0.25) (layer "F.Cu") (net 10))
   (segment (start 142.8206 83.0326) (end 134.7724 83.0326) (width 0.25) (layer "F.Cu") (net 10))
   (segment (start 134.518 92.8518) (end 134.518 97.669) (width 0.25) (layer "F.Cu") (net 10))
   (segment (start 154.2898 89.7636) (end 156.4488 87.6046) (width 0.25) (layer "F.Cu") (net 10))
-  (segment (start 134.493 89.5832) (end 135.6742 89.5832) (width 0.25) (layer "F.Cu") (net 10))
   (segment (start 148.9244 91.827) (end 150.9878 89.7636) (width 0.25) (layer "F.Cu") (net 10))
   (segment (start 154.4809 84.5312) (end 155.8138 84.5312) (width 0.25) (layer "F.Cu") (net 10))
@@
   (segment (start 156.7282 84.5312) (end 156.9568 84.5312) (width 0.25) (layer "F.Cu") (net 10))
   (segment (start 147.68 91.827) (end 148.9244 91.827) (width 0.25) (layer "F.Cu") (net 10))
+  (segment (start 135.6742 89.5832) (end 135.668 89.577) (width 0.25) (layer "F.Cu") (net 10))
   (segment (start 156.4488 84.8106) (end 156.7282 84.5312) (width 0.25) (layer "F.Cu") (net 10))
-  (segment (start 135.6742 89.5832) (end 135.668 89.577) (width 0.25) (layer "F.Cu") (net 10))
   (segment (start 158.5976 84.5312) (end 162.3568 88.2904) (width 0.25) (layer "F.Cu") (net 10))
   (segment (start 163.5608 91.288101) (end 163.5608 89.4944) (width 0.25) (layer "F.Cu") (net 10))
@@
   (segment (start 156.1948 99.404899) (end 156.1948 94.3356) (width 0.25) (layer "F.Cu") (net 22))
   (segment (start 143.11 86.2038) (end 144.7648 87.8586) (width 0.25) (layer "F.Cu") (net 22))
+  (segment (start 159.5222 91.44) (end 160.6398 92.5576) (width 0.25) (layer "F.Cu") (net 22))
+  (segment (start 159.2815 91.44) (end 159.5222 91.44) (width 0.25) (layer "F.Cu") (net 22))
   (segment (start 160.6398 92.5474) (end 162.3568 90.8304) (width 0.25) (layer "F.Cu") (net 22))
   (segment (start 157.246058 100.456157) (end 156.1948 99.404899) (width 0.25) (layer "F.Cu") (net 22))
   (segment (start 160.6398 92.5576) (end 160.6398 92.5474) (width 0.25) (layer "F.Cu") (net 22))
-  (segment (start 159.2815 91.44) (end 161.7472 91.44) (width 0.25) (layer "F.Cu") (net 22))
   (segment (start 161.7472 91.44) (end 162.3568 90.8304) (width 0.25) (layer "F.Cu") (net 22))
   (via (at 156.1948 94.3356) (size 0.8) (drill 0.4) (layers "F.Cu" "B.Cu") (net 22))

Commit message: COmpleted with silkscreen and footprints(logo).
Parts:
- added REF**: KiCad-Logo2_5mm_SilkScreen, Symbol:KiCad-Logo2_5mm_SilkScreen, B.Cu at (142.6, 87.7)
- moved R2 1.74 mm to (128.9, 102.1)
- moved R3 1.52 mm to (131.9, 102.1)
Connections:
- BT1 pad 1: Net-(BT1-+) -> /VCC
- C5 pad 1: Net-(BT1-+) -> /VCC
- R5 pad 1: Net-(BT1-+) -> /VCC
- U3 pad 18: Net-(BT1-+) -> /VCC
- U3 pad 6: Net-(BT1-+) -> /VCC
Routing:
- net Net-(BT1-+): track 61.7 -> 0.00 mm, vias 1 -> 0
- net /VCC: track 157.3 -> 218.7 mm, vias 8 -> 9
- net Net-(U4-~{INTA}): track 10.3 -> 8.93 mm
- net Net-(U4-SQW/~INT): track 7.18 -> 5.84 mm
Other:
- board text added: "+ GND"
- board text added: "ATMEGA328P-AU"
- board text added: "Created by Kunj Chauhan"
- board text added: "D2"
- board text added: "D3"
- board text added: "D4"
- board text added: "D5"
- board text added: "D6"
- board text added: "D7"
- board text added: "D8"
- board text added: "GND"
- board text added: "I2C"
- board text added: "ICSP"
- board text added: "MCU Datalogger -2Mb EEPROOM -RTC -I2C,SPI,GPIO"
- board text added: "MISO"
- board text added: "MOSI"
- board text added: "RST"
- board text added: "RX"
- board text added: "SCK"
- board text added: "SDA"
- board text added: "TX"
- board text added: "UART"
- board text added: "VCC"
