File: Atmega328p_board.kicad_sch (KiCad schematic)
At the start: 25 parts, among them U1 24LC1025, U2 24LC1025, U3 ATMEGA328P-AU, U4 DS1337S_, Y1 16MHz, Y2 32.768 KHz

Commit message: 4 layer pcb fixed with changes of sck and scl
Connections:
- net SCK: no longer R6.2, U1.6 (SCL), U2.6 (SCL), U3.28 (PC5), U4.6 (SCL)
- new net SCL: R6.2, U1.6 (SCL), U2.6 (SCL), U3.28 (PC5), U4.6 (SCL)
Other:
- sheet connector ports: added SCL; removed none
Changed lines of the file:
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@@
+    (stroke (width 0) (type default))
+  )
+  (wire (pts (xy 143.51 123.19) (xy 146.685 123.19))
     (stroke (width 0) (type default))
   )
@@
     (effects (font (size 1.27 1.27)) (justify left bottom))
   )
-  (label "SCK" (at 95.25 173.99 0) (fields_autoplaced)
+  (label "SCL" (at 95.25 173.99 0) (fields_autoplaced)
     (effects (font (size 1.27 1.27)) (justify left bottom))
   )
@@
     (effects (font (size 1.27 1.27)) (justify left bottom))
   )
-  (label "SCK" (at 83.82 166.37 0) (fields_autoplaced)
+  (label "SCL" (at 83.82 166.37 0) (fields_autoplaced)
     (effects (font (size 1.27 1.27)) (justify left bottom))
   )
@@
     (effects (font (size 1.27 1.27)) (justify left bottom))
   )
-  (label "SCK" (at 46.355 62.23 0) (fields_autoplaced)
+  (label "SCL" (at 46.355 62.23 0) (fields_autoplaced)
     (effects (font (size 1.27 1.27)) (justify left bottom))
   )
@@
     (effects (font (size 1.27 1.27)) (justify left bottom))
   )
-  (label "SCK" (at 185.42 74.93 180) (fields_autoplaced)
+  (label "SCL" (at 185.42 74.93 180) (fields_autoplaced)
     (effects (font (size 1.27 1.27)) (justify right bottom))
   )
@@
     (effects (font (size 1.27 1.27)) (justify right bottom))
   )
+  (label "SCL" (at 143.51 123.19 180) (fields_autoplaced)
+    (effects (font (size 1.27 1.27)) (justify right bottom))
+  )
   (label "SDA" (at 83.82 163.83 0) (fields_autoplaced)
     (effects (font (size 1.27 1.27)) (justify left bottom))
@@
     (effects (font (size 1.27 1.27)) (justify left bottom))
   )
-  (label "SCK" (at 49.53 166.37 0) (fields_autoplaced)
+  (label "SCL" (at 49.53 166.37 0) (fields_autoplaced)
     (effects (font (size 1.27 1.27)) (justify left bottom))
   )
@@
       (effects (font (size 1.27 1.27)) (justify left))
     )
+    (pin "SCL" passive (at 146.685 123.19 180)
+      (effects (font (size 1.27 1.27)) (justify left))
+    )
